File: adapter/adapter.kicad_pcb (KiCad board)
At the start: 2 copper layers, 101.7 x 36.7 mm, 14 parts, among them J1 AudioJack4, J2 AudioJack4, J3 Conn_01x02_Female, J4 Conn_01x03_Female, J5 Conn_01x03_Female, J6 Conn_01x02_Female, SW1 SW_SPST, SW2 SW_SPST, U1 ProMicro, U2 ProMicro

Commit message: left adapter
Parts:
- added J7: Conn_01x06_Female, Connector_PinHeader_2.54mm:PinHeader_1x06_P2.54mm_Vertical, F.Cu at (120.9, 31.5)
- added J9: Conn_01x06_Female, Connector_PinHeader_2.54mm:PinHeader_1x06_P2.54mm_Vertical, F.Cu at (195.8, 32.3)
- U1: value ProMicro -> eliteC; footprint customs:Elite-C -> Library:Elite-C-castellated-29pin-holes
- U2: value ProMicro -> eliteC; footprint footprints:Elite-C -> Library:Elite-C-castellated-29pin-holes
- moved J6 8.87 mm to (200.3, 31.2)
- moved J3 8.74 mm to (115.4, 31.1)
Connections:
- J1 pad S: Net-(J1-PadS) -> unconnected-(J1-PadS)
- J2 pad S: Net-(J2-PadS) -> unconnected-(J2-PadS)
- J3 pad 1: Net-(J1-PadR2) -> Net-(J3-Pad1)
- J6 pad 1: Net-(J2-PadR2) -> Net-(J6-Pad1)
- U1 pad 1: Net-(U1-Pad1) -> Din
- U1 pad 19: Net-(U1-Pad19) -> unconnected-(U1-Pad19)
- U1 pad 2: Din -> Net-(J1-PadR2)
- U1 pad 20: Net-(U1-Pad20) -> unconnected-(U1-Pad20)
- U1 pad 24: Net-(U1-Pad24) -> ss
- U1 pad 6: Net-(J1-PadR2) -> Net-(J3-Pad1)
- U2 pad 1: Net-(U2-Pad1) -> Din2
- U2 pad 19: Net-(U2-Pad19) -> unconnected-(U2-Pad19)
- U2 pad 2: Din2 -> Net-(J2-PadR2)
- U2 pad 20: Net-(U2-Pad20) -> unconnected-(U2-Pad20)
- U2 pad 24: Net-(U2-Pad24) -> ss2
- U2 pad 6: Net-(J2-PadR2) -> Net-(J6-Pad1)
Routing:
- net Vcc2: track 81.0 -> 0.00 mm
- net Gnd2: track 39.3 -> 0.00 mm
- net Rst: track 60.7 -> 23.9 mm, vias 0 -> 2
- net Net-(J2-PadR2): track 31.8 -> 0.00 mm
- net ss: track 0.00 -> 29.8 mm
- net Din2: track 28.6 -> 0.00 mm
- net Net-(J3-Pad1): track 0.00 -> 25.8 mm, vias 0 -> 1
- net Din: track 58.5 -> 35.2 mm
- net Net-(J1-PadR2): track 55.8 -> 36.6 mm, vias 0 -> 1
- net Rst2: track 13.4 -> 0.00 mm
- net Net-(J6-Pad2): track 12.8 -> 0.00 mm
- net mosi: track 0.00 -> 6.43 mm
- net Net-(J3-Pad2): track 29.8 -> 25.1 mm, vias 0 -> 1
- net sc: track 0.00 -> 4.46 mm
- net miso: track 0.00 -> 4.46 mm
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Other:
- outline, holes or cut-outs redrawn
- board text added: "Charybdis adapter 1.0"
- board text added: "Trackball"
- board text added: "miso"
- board text added: "mosi"
- board text added: "sc"
- board text added: "ss"
- board text removed: "MCU adapter 1.4"
