File: adapter/adapter.kicad_pcb (KiCad board)
At the start: 2 copper layers, 101.7 x 36.7 mm, 16 parts, among them J1 AudioJack4, J2 AudioJack4, J3 Conn_01x02_Female, J4 Conn_01x03_Female, J5 Conn_01x03_Female, J6 Conn_01x02_Female, J7 Conn_01x06_Female, J9 Conn_01x06_Female, SW1 SW_SPST, SW2 SW_SPST, U1 eliteC, U2 eliteC

Commit message: routing
Parts:
- moved J9 1.16 mm to (194.9, 31.5)
Routing:
- net Vcc2: track 0.00 -> 92.8 mm
- net Gnd2: track 0.00 -> 75.9 mm, vias 0 -> 2
- net sc2: track 0.00 -> 48.5 mm, vias 0 -> 1
- net miso2: track 0.00 -> 36.5 mm
- net mosi2: track 0.00 -> 36.0 mm
- net Din2: track 0.00 -> 32.9 mm
- net ss2: track 0.00 -> 29.5 mm
- net Rst2: track 0.00 -> 15.0 mm, vias 0 -> 1
- net Net-(J2-PadR2): track 0.00 -> 12.0 mm
- net Net-(J6-Pad2): track 0.00 -> 9.55 mm, vias 0 -> 1
- net Net-(J6-Pad1): track 0.00 -> 9.55 mm, vias 0 -> 1
- net Gnd: track 56.6 -> 64.2 mm, vias 0 -> 1
Other:
- outline, holes or cut-outs redrawn
