File: adapter/adapter.kicad_pcb (KiCad board)
At the start: 2 copper layers, 101.7 x 36.7 mm, 16 parts, among them J1 AudioJack4, J2 AudioJack4, J3 Conn_01x02_Female, J4 Conn_01x03_Female, J5 Conn_01x03_Female, J6 Conn_01x02_Female, J7 Conn_01x06_Female, J9 Conn_01x06_Female, SW1 SW_SPST, SW2 SW_SPST, U1 eliteC, U2 eliteC

Commit message: silkscreen
Other:
- board text added: "Left"
- board text added: "Right"
Changed lines of the file:
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@@
     (effects (font (size 1 1) (thickness 0.15)))
   )
-  (gr_text "ss" (at 197.052 33.704 45) (layer "F.SilkS")
+  (gr_text "ss" (at 197.03 33.68 45) (layer "F.SilkS")
     (effects (font (size 1 1) (thickness 0.15)))
   )
@@
     (effects (font (size 1 1) (thickness 0.15)))
   )
+  (gr_text "Right" (at 142.38 38.19 270) (layer "F.SilkS")
+    (effects (font (size 1.2 1.2) (thickness 0.2)))
+  )
   (gr_text "sc" (at 118.89 38.44 -45) (layer "F.SilkS")
     (effects (font (size 1 1) (thickness 0.15)))
@@
     (effects (font (size 1 1) (thickness 0.15)))
   )
-  (gr_text "sc" (at 196.798 38.784 45) (layer "F.SilkS")
+  (gr_text "sc" (at 196.798 38.67 45) (layer "F.SilkS")
     (effects (font (size 1 1) (thickness 0.15)))
   )
@@
     (effects (font (size 1 1) (thickness 0.15)))
   )
+  (gr_text "Left" (at 172.5 37.47 90) (layer "F.SilkS")
+    (effects (font (size 1.2 1.2) (thickness 0.2)))
+  )
   (gr_text "D1" (at 113.275 28.115 -45) (layer "F.SilkS")

Commit message: silkscreen
Other:
- board text added: "Charybdis adapter 1.1"
- board text added: "DIN"
- board text added: "GND"
- board text added: "MISO"
- board text added: "MOSI"
- board text added: "SC"
- board text added: "SCK"
- board text added: "SS"
- board text added: "VCC"
- board text removed: "Charybdis adapter 1.0"
- board text removed: "Din"
- board text removed: "miso"
- board text removed: "mosi"
- board text removed: "sc"
- board text removed: "ss"
Changed lines of the file:
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@@
       (viasonmask false)
       (mode 1)
-      (useauxorigin false)
+      (useauxorigin true)
       (hpglpennumber 1)
       (hpglpenspeed 20)
@@
   (gr_line (start 120.306081 47.519414) (end 120.316257 47.662099) (layer "F.Fab") (width 0.2))
   (gr_text "RST" (at 143.8 34.05) (layer "B.SilkS")
-    (effects (font (size 1 1) (thickness 0.15)) (justify mirror))
+    (effects (font (size 0.8 0.8) (thickness 0.2)) (justify mirror))
   )
   (gr_text "RST" (at 172.1 34.2) (layer "B.SilkS")
-    (effects (font (size 1 1) (thickness 0.15)) (justify mirror))
+    (effects (font (size 0.8 0.8) (thickness 0.2)) (justify mirror))
   )
   (gr_text "S" (at 117.3 15.6) (layer "F.SilkS")
+    (effects (font (size 0.8 0.8) (thickness 0.15)))
+  )
+  (gr_text "Charybdis adapter 1.1" (at 130.8 48.5) (layer "F.SilkS")
     (effects (font (size 1 1) (thickness 0.15)))
   )
-  (gr_text "Charybdis adapter 1.0" (at 130.8 48.5) (layer "F.SilkS")
-    (effects (font (size 1 1) (thickness 0.15)))
-  )
   (gr_text "D0" (at 141.39 28.92) (layer "F.SilkS")
     (effects (font (size 0.8 0.8) (thickness 0.15)))
   )
-  (gr_text "Vcc" (at 202.72 33.44 45) (layer "F.SilkS")
-    (effects (font (size 1 1) (thickness 0.15)))
-  )
-  (gr_text "Gnd" (at 200.1 18.5) (layer "F.SilkS")
-    (effects (font (size 1 1) (thickness 0.15)))
-  )
-  (gr_text "Vcc" (at 200 22.6) (layer "F.SilkS")
-    (effects (font (size 1 1) (thickness 0.15)))
-  )
-  (gr_text "ss" (at 197.03 33.68 45) (layer "F.SilkS")
-    (effects (font (size 1 1) (thickness 0.15)))
-  )
-  (gr_text "ss" (at 118.76 33.18 -45) (layer "F.SilkS")
-    (effects (font (size 1 1) (thickness 0.15)))
-  )
-  (gr_text "mosi" (at 118.15 35.3 -45) (layer "F.SilkS")
-    (effects (font (size 1 1) (thickness 0.15)))
+  (gr_text "VCC" (at 202.72 33.44 45) (layer "F.SilkS")
+    (effects (font (size 0.8 0.8) (thickness 0.15)))
+  )
+  (gr_text "Gnd" (at 200.057143 18.5) (layer "F.SilkS")
+    (effects (font (size 0.8 0.8) (thickness 0.15)))
+  )
+  (gr_text "Vcc" (at 200.152381 22.6) (layer "F.SilkS")
+    (effects (font (size 0.8 0.8) (thickness 0.15)))
+  )
+  (gr_text "SS" (at 197.115127 33.2092 45) (layer "F.SilkS")
+    (effects (font (size 0.8 0.8) (thickness 0.15)))
+  )
+  (gr_text "SS" (at 118.769374 33.140001 -45) (layer "F.SilkS")
+    (effects (font (size 0.8 0.8) (thickness 0.15)))
+  )
+  (gr_text "MOSI" (at 118.230626 35.68 -45) (layer "F.SilkS")
+    (effects (font (size 0.8 0.8) (thickness 0.15)))
   )
   (gr_text "S" (at 200.8 15.6) (layer "F.SilkS")
-    (effects (font (size 1 1) (thickness 0.15)))
-  )
-  (gr_text "Gnd" (at 118.4 43.55 -45) (layer "F.SilkS")
-    (effects (font (size 1 1) (thickness 0.15)))
+    (effects (font (size 0.8 0.8) (thickness 0.15)))
+  )
+  (gr_text "GND" (at 118.432656 43.3 -45) (layer "F.SilkS")
+    (effects (font (size 0.8 0.8) (thickness 0.15)))
   )
   (gr_text "D1" (at 202.7 28.17 45) (layer "F.SilkS")
-    (effects (font (size 1 1) (thickness 0.15)))
+    (effects (font (size 0.8 0.8) (thickness 0.15)))
   )
   (gr_text "B0" (at 122.185 16.164) (layer "F.SilkS")
     (effects (font (size 0.8 0.8) (thickness 0.15)))
   )
-  (gr_text "Gnd" (at 197.56 43.61 45) (layer "F.SilkS")
-    (effects (font (size 1 1) (thickness 0.15)))
-  )
-  (gr_text "Gnd" (at 202.59 35.97 45) (layer "F.SilkS")
-    (effects (font (size 1 1) (thickness 0.15)))
-  )
-  (gr_text "Din" (at 112.985 37.965 -45) (layer "F.SilkS")
-    (effects (font (size 1 1) (thickness 0.15)))
-  )
-  (gr_text "Vcc" (at 116.4 22.6) (layer "F.SilkS")
-    (effects (font (size 1 1) (thickness 0.15)))
-  )
-  (gr_text "mosi" (at 197.56 35.482 45) (layer "F.SilkS")
-    (effects (font (size 1 1) (thickness 0.15)))
+  (gr_text "GND" (at 197.438375 43.572401 45) (layer "F.SilkS")
+    (effects (font (size 0.8 0.8) (thickness 0.15)))
+  )
+  (gr_text "GND" (at 202.59 35.97 45) (layer "F.SilkS")
+    (effects (font (size 0.8 0.8) (thickness 0.15)))
+  )
+  (gr_text "DIN" (at 112.985 37.965 -45) (layer "F.SilkS")
+    (effects (font (size 0.8 0.8) (thickness 0.15)))
+  )
+  (gr_text "VCC" (at 116.538096 22.6) (layer "F.SilkS")
+    (effects (font (size 0.8 0.8) (thickness 0.15)))
+  )
+  (gr_text "MOSI" (at 197.6 35.8 45) (layer "F.SilkS")
+    (effects (font (size 0.8 0.8) (thickness 0.15)))
   )
   (gr_text "D0" (at 113.175 30.515 -45) (layer "F.SilkS")
-    (effects (font (size 1 1) (thickness 0.15)))
-  )
-  (gr_text "Vcc" (at 118.65 30.85 -45) (layer "F.SilkS")
-    (effects (font (size 1 1) (thickness 0.15)))
-  )
-  (gr_text "miso" (at 197.56 40.562 45) (layer "F.SilkS")
-    (effects (font (size 1 1) (thickness 0.15)))
+    (effects (font (size 0.8 0.8) (thickness 0.15)))
+  )
+  (gr_text "VCC" (at 118.5 30.6 -45) (layer "F.SilkS")
+    (effects (font (size 0.8 0.8) (thickness 0.15)))
+  )
+  (gr_text "MISO" (at 197.6 40.9816 45) (layer "F.SilkS")
+    (effects (font (size 0.8 0.8) (thickness 0.15)))
   )
   (gr_text "Right" (at 142.38 38.19 270) (layer "F.SilkS")
     (effects (font (size 1.2 1.2) (thickness 0.2)))
   )
-  (gr_text "sc" (at 118.89 38.44 -45) (layer "F.SilkS")
-    (effects (font (size 1 1) (thickness 0.15)))
+  (gr_text "SCK" (at 118.526938 38.22 -45) (layer "F.SilkS")
+    (effects (font (size 0.8 0.8) (thickness 0.15)))
   )
   (gr_text "B0" (at 122.2 68.279) (layer "F.SilkS")
     (effects (font (size 0.8 0.8) (thickness 0.15)))
   )
-  (gr_text "miso" (at 118.4 40.48 -45) (layer "F.SilkS")
-    (effects (font (size 1 1) (thickness 0.15)))
-  )
-  (gr_text "sc" (at 196.798 38.67 45) (layer "F.SilkS")
-    (effects (font (size 1 1) (thickness 0.15)))
-  )
-  (gr_text "Vcc" (at 112.98 32.97 -45) (layer "F.SilkS")
-    (effects (font (size 1 1) (thickness 0.15)))
-  )
-  (gr_text "Serial" (at 115.999998 26.45) (layer "F.SilkS")
-    (effects (font (size 1 1) (thickness 0.15)))
+  (gr_text "MISO" (at 118.230626 40.76 -45) (layer "F.SilkS")
+    (effects (font (size 0.8 0.8) (thickness 0.15)))
+  )
+  (gr_text "SC" (at 197.128595 38.390801 45) (layer "F.SilkS")
+    (effects (font (size 0.8 0.8) (thickness 0.15)))
+  )
+  (gr_text "VCC" (at 112.98 32.97 -45) (layer "F.SilkS")
+    (effects (font (size 0.8 0.8) (thickness 0.15)))
+  )
+  (gr_text "Serial" (at 115.4 26.5) (layer "F.SilkS")
+    (effects (font (size 0.8 0.8) (thickness 0.2)))
   )
   (gr_text "D0" (at 202.76 30.85 45) (layer "F.SilkS")
-    (effects (font (size 1 1) (thickness 0.15)))
+    (effects (font (size 0.8 0.8) (thickness 0.15)))
   )
   (gr_text "B0" (at 174.3 16.079) (layer "F.SilkS")
@@
   )
   (gr_text "RGB" (at 115.4 41.2) (layer "F.SilkS")
-    (effects (font (size 1.2 1.2) (thickness 0.2)))
-  )
-  (gr_text "Gnd" (at 112.85 35.5 -45) (layer "F.SilkS")
-    (effects (font (size 1 1) (thickness 0.15)))
+    (effects (font (size 0.8 0.8) (thickness 0.2)))
+  )
+  (gr_text "GND" (at 112.85 35.5 -45) (layer "F.SilkS")
+    (effects (font (size 0.8 0.8) (thickness 0.15)))
   )
   (gr_text "Trackball" (at 120.9 46.4) (layer "F.SilkS")
-    (effects (font (size 1 1) (thickness 0.15)))
-  )
-  (gr_text "Vcc" (at 197.306 30.656 45) (layer "F.SilkS")
-    (effects (font (size 1 1) (thickness 0.15)))
+    (effects (font (size 0.8 0.8) (thickness 0.2)))
+  )
+  (gr_text "VCC" (at 197.384501 30.618401 45) (layer "F.SilkS")
+    (effects (font (size 0.8 0.8) (thickness 0.15)))
   )
   (gr_text "Left" (at 172.5 37.47 90) (layer "F.SilkS")
@@
   )
   (gr_text "D1" (at 113.275 28.115 -45) (layer "F.SilkS")
-    (effects (font (size 1 1) (thickness 0.15)))
-  )
-  (gr_text "Charybdis adapter 1.0" (at 185.85 48.25) (layer "F.SilkS")
+    (effects (font (size 0.8 0.8) (thickness 0.15)))
+  )
+  (gr_text "Charybdis adapter 1.1" (at 185.85 48.25) (layer "F.SilkS")
     (effects (font (size 1 1) (thickness 0.15)))
   )
@@
   )
   (gr_text "RGB" (at 200.4 41.373) (layer "F.SilkS")
-    (effects (font (size 1.2 1.2) (thickness 0.2)))
-  )
-  (gr_text "Din" (at 202.55 38.45 45) (layer "F.SilkS")
-    (effects (font (size 1 1) (thickness 0.15)))
-  )
-  (gr_text "Serial" (at 199.449998 26.2475) (layer "F.SilkS")
-    (effects (font (size 1 1) (thickness 0.15)))
+    (effects (font (size 0.8 0.8) (thickness 0.2)))
+  )
+  (gr_text "DIN" (at 202.55 38.45 45) (layer "F.SilkS")
+    (effects (font (size 0.8 0.8) (thickness 0.15)))
+  )
+  (gr_text "Serial" (at 200.2 26.6) (layer "F.SilkS")
+    (effects (font (size 0.8 0.8) (thickness 0.2)))
   )
   (gr_text "Trackball" (at 196.7 46.22) (layer "F.SilkS")
-    (effects (font (size 1 1) (thickness 0.15)))
-  )
-  (gr_text "Gnd" (at 116.385 18.8) (layer "F.SilkS")
-    (effects (font (size 1 1) (thickness 0.15)))
+    (effects (font (size 0.8 0.8) (thickness 0.2)))
+  )
+  (gr_text "GND" (at 116.461905 18.8) (layer "F.SilkS")
+    (effects (font (size 0.8 0.8) (thickness 0.15)))
   )
   (gr_text "Install \nElite-C,\ncables\nand jack\non this\nside" (at 184.1 23.15) (layer "F.SilkS")

Commit message: slikscreen
Parts:
- added G***: LOGO, LOGO, F.Cu at (123.9, 58.3)
- added G***: LOGO, LOGO, B.Cu at (124.0, 58.3)
- added G***: LOGO, LOGO, B.Cu at (102.0, 29.2)
- added G***: LOGO, LOGO, B.Cu at (146.1, 29.2)
- moved J2 38.4 mm to (164.5, 29.4)
- moved J5 38.4 mm to (162.5, 40.8)
- moved J6 38.4 mm to (162.4, 38.1)
- moved J9 38.4 mm to (157.1, 38.4)
- moved REF** 38.4 mm to (132.2, 25.2)
- moved SW2 38.4 mm to (134.1, 35.8)
- moved REF** 38.4 mm to (166.7, 53.0)
- moved U2 38.4 mm to (146.2, 37.0)
- moved J7 30.5 mm to (91.2, 38.4)
- moved U1 30.5 mm to (102.2, 37.1)
- moved J1 30.5 mm to (89.1, 29.3)
- moved J3 30.5 mm to (85.6, 38.0)
- moved J4 30.5 mm to (85.6, 40.8)
- moved REF** 30.5 mm to (116.0, 25.2)
- moved REF** 30.5 mm to (81.4, 53.1)
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Other:
- board size 101.7 x 36.7 mm -> 93.8 x 42.3 mm
- board text added: "2021 QUENTIN LEBASTARD"
- board text added: "BASTARDKB.COM"
- board text added: "CHARYBDIS HOLDER"
- board text added: "GITHUB.COM/BASTARDKB"
- board text added: "Have a fun build"
- board text added: "LEFT"
- board text added: "REV 1.2"
- board text added: "RIGHT"
- board text added: "SERIAL"
- board text added: "TRACKBALL"
- board text removed: "Charybdis adapter 1.1"
- board text removed: "Left"
- board text removed: "Right"
- board text removed: "Serial"
- board text removed: "Trackball"

Commit message: routing
Routing:
- net miso2: track 36.5 -> 52.4 mm
- net sc2: track 48.5 -> 41.4 mm, vias 1 -> 0
- net Vcc2: track 92.8 -> 98.1 mm
- net Gnd2: track 75.9 -> 80.1 mm
Other:
- board text added: "REV 1.21"
- board text removed: "REV 1.2"
